Commit message: Update URDF with correct robot structure

File: urdf/exam_robot.urdf (robot description, URDF)
Before this commit: robot exam_robot, 4 links, 3 joints
Links:
- link sensor_link: mass 0.1 -> 0.05; geometry collision box size=0.05 0.05 0.05; visual box size=0.05 0.05 0.05
Joints:
- joint base_to_left_wheel: origin xyz=-0.1 0.17 0 rpy=1.5708 0 0 -> xyz=-0.1 0.17 0 rpy=0 0 0
- joint base_to_right_wheel: origin xyz=-0.1 -0.17 0 rpy=1.5708 0 0 -> xyz=-0.1 -0.17 0 rpy=0 0 0
- joint base_to_sensor: origin xyz=0.2 0 0.05 rpy=0 0 0 -> xyz=0.2 0 0.08 rpy=0 0 0
